File: Hardware/Placa_PCB/Power.kicad_sch (KiCad schematic)
At the start: 13 parts, among them J2 USB_C_Receptacle_PowerOnly_6P, J3 USB_C_Receptacle_USB2.0_16P, Q4 DMG2305UX-7

Commit message: Update ESP32 MCU schematic and connections
Changed lines of the file:
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@@
-	)
-	(junction
-		(at 224.79 105.41)
-		(diameter 0)
-		(color 0 0 0 0)
 	)
 	(junction
@@
 	(wire
 		(pts
-			(xy 224.79 105.41) (xy 233.68 105.41)
-		)
-		(stroke
-			(width 0)
-			(type default)
-		)
-	)
-	(wire
-		(pts
 			(xy 177.8 77.47) (xy 182.88 77.47)
 		)
@@
 	(wire
 		(pts
-			(xy 224.79 105.41) (xy 224.79 106.68)
-		)
-		(stroke
-			(width 0)
-			(type default)
-		)
-	)
-	(wire
-		(pts
 			(xy 171.45 74.93) (xy 171.45 77.47)
 		)
@@
 	(wire
 		(pts
-			(xy 224.79 104.14) (xy 224.79 105.41)
+			(xy 224.79 104.14) (xy 224.79 106.68)
 		)
 		(stroke
@@
 	)
 	(label "V_USB_PROG"
-		(at 224.79 71.12 180)
+		(at 224.79 71.12 0)
 		(effects
 			(font
 				(size 1.27 1.27)
 			)
-			(justify right bottom)
+			(justify left bottom)
 		)
 	)
@@
 		(polyline
 			(pts
-				(xy 209.55 59.69) (xy 209.55 121.92) (xy 265.43 121.92) (xy 265.43 59.69)
+				(xy 209.55 55.88) (xy 209.55 121.92) (xy 265.43 121.92) (xy 265.43 55.88)
 			)
 			(stroke
@@
 		(polyline
 			(pts
-				(xy 111.76 59.69) (xy 111.76 121.92) (xy 203.2 121.92) (xy 203.2 59.69)
+				(xy 111.76 55.88) (xy 111.76 121.92) (xy 203.2 121.92) (xy 203.2 55.88)
 			)
 			(stroke
@@
 		(polyline
 			(pts
-				(xy 27.94 59.69) (xy 105.41 59.69) (xy 105.41 121.92) (xy 27.94 121.92)
+				(xy 27.305 55.88) (xy 104.775 55.88) (xy 105.41 121.92) (xy 27.94 121.92)
 			)
 			(stroke
@@
 					(unit 1)
 				)
-			)
-		)
-	)
-	(symbol
-		(lib_id "power:PWR_FLAG")
-		(at 233.68 105.41 270)
-		(unit 1)
-		(exclude_from_sim no)
-		(in_bom yes)
-		(on_board yes)
-		(dnp no)
-		(fields_autoplaced yes)
-		(property "Reference" "#FLG02"
-			(at 235.585 105.41 0)
-			(effects
-				(font
-					(size 1.27 1.27)
-				)
-				(hide yes)
-			)
-		)
-		(property "Value" "PWR_FLAG"
-			(at 237.49 105.4099 90)
-			(effects
-				(font
-					(size 1.27 1.27)
-				)
-				(justify left)
-			)
-		)
-		(property "Footprint" ""
-			(at 233.68 105.41 0)
-			(effects
-				(font
-					(size 1.27 1.27)
-				)
-				(hide yes)
-			)
-		)
-		(property "Datasheet" "~"
-			(at 233.68 105.41 0)
-			(effects
-				(font
-					(size 1.27 1.27)
-				)
-				(hide yes)
-			)
-		)
-		(property "Description" "Special symbol for telling ERC where power comes from"
-			(at 233.68 105.41 0)
-			(effects
-				(font
-					(size 1.27 1.27)
-				)
-				(hide yes)
-			)
-		)
-		(pin "1"
-		)
-		(instances
-			(project "ScramblerBot"
-				(path "/ca162c4b-e7f6-494c-9ea1-0d86ef4a8e44/bb166e8a-7d54-4ae8-a0b2-867dec2483b7"
-					(reference "#FLG02")
-					(unit 1)
-				)
